File: ESP32_GRBL_SUBD/ESP32_GRBL_SUBD.kicad_pcb (KiCad board)
At the start: 2 copper layers, 91 x 67 mm, 83 parts, among them J1 DB25_Female_MountingHoles, J10 Screw_Terminal_01x02, J11 Screw_Terminal_01x02, J12 Screw_Terminal_01x02, J13 Screw_Terminal_01x02, J14 Screw_Terminal_01x02, J2 Micro_SD_Card, J3 Conn_01x19_Female, J3a1 Conn_01x19_Female, J4 Conn_01x19_Female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

Commit message: changed value of Resistor to match my actual soldered PCB
Parts:
- R41: value dnp -> 0R
Changed lines of the file:
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@@
       (effects (font (size 1 1) (thickness 0.15)) (justify mirror))
     )
-    (fp_text value "dnp" (at 0 -1.43) (layer "B.Fab")
+    (fp_text value "0R" (at 0 -1.43) (layer "B.Fab")
       (effects (font (size 1 1) (thickness 0.15)) (justify mirror))
     )
